File: hardware_design/pcb_design/bldc_driver_fpga/3PH_INVERTER.kicad_sch (KiCad schematic)
At the start: 24 parts, among them IC1 DRV8300NRGE, Q1 CSD17578Q5A, Q2 CSD17578Q5A, Q3 CSD17578Q5A, Q4 CSD17578Q5A, Q5 CSD17578Q5A, Q6 CSD17578Q5A

Commit message: Implemented pure sinewave drive from programmable logic. Set up time base generator for ADC.
Parts:
- added C15, C18: 0.1uF 16V, Capacitor_SMD:C_0603_1608Metric_Pad1.08x0.95mm_HandSolder, symbol Device:C_Small
- added C16, C19: 470pF 16V, Capacitor_SMD:C_0603_1608Metric_Pad1.08x0.95mm_HandSolder, symbol Device:C_Small
- added D10, D8, D9: MBR0580, Diode_SMD:D_SOD-123F, symbol Device:D_Schottky_Small
- added D5: 1V, Package_TO_SOT_SMD:SOT-23, symbol Device:D_Zener_Small
- added IC2: INA2181A2IDSQR, bldc_driver_fpga:WSON-10-1EP_2.0x2.0mm_P0.4mm_EP0.9x1.5mm, symbol driver_lib_kicad6:INA2181A2IDSQR
- added R15: 2.2k, Resistor_SMD:R_0603_1608Metric_Pad0.98x0.95mm_HandSolder, symbol Device:R_Small
- added R16, R29: 0.02R, Resistor_SMD:R_1206_3216Metric_Pad1.30x1.75mm_HandSolder, symbol Device:R_Small
- C10, C11, C9: footprint Capacitor_SMD:C_0603_1608Metric_Pad1.05x0.95mm_HandSolder -> Capacitor_SMD:C_0603_1608Metric_Pad1.08x0.95mm_HandSolder
- C8: footprint Capacitor_SMD:C_0805_2012Metric_Pad1.15x1.40mm_HandSolder -> Capacitor_SMD:C_0603_1608Metric_Pad1.08x0.95mm_HandSolder
- IC1: footprint Package_DFN_QFN:VQFN-24-1EP_4x4mm_P0.5mm_EP2.45x2.45mm_ThermalVias -> bldc_driver_fpga:VQFN-24-1EP_4x4mm_P0.5mm_EP2.45x2.45mm_ThermalViasBig
- Q1, Q3, Q5: footprint bldc_driver_fpga:TDSON-8-1_HandSoldering_SGD -> bldc_driver_fpga:TDSON-8-1_HandSolderingVias_SGD
Connections:
- net Phase A Current Sense/LS_SOURCE is gone; now on net PGND: Q2.1 (S)
- net sheet613E4E23/LS_SOURCE is gone; now on net PGND: Q4.1 (S)
- net DGND: now also C15.2, C16.1, C18.2, C19.1, D5.2 (A), IC2.11 (EP), IC2.4 (GND); no longer C8.2, IC1.25 (EP), IC1.6 (GND), R8.2
- net IS_U: now also IC2.1 (OUT)
- net IS_V: now also IC2.9 (OUT)
- net IVDD: now also C15.1, IC2.10 (VS), R15.1
- net PGND: now also C8.2, IC1.25 (EP), IC1.6 (GND), R8.2, C16.2, C19.2, D10.2 (A), D8.2 (A), D9.2 (A)
- net U_OUT: now also D10.1 (K), IC2.2 (INN), R16.2; no longer C9.1, IC1.18 (SHA), Q1.1 (S), Q2.3 (D)
- net V_OUT: now also D9.1 (K), IC2.8 (INN), R29.2; no longer C10.1, IC1.15 (SHB), Q3.1 (S), Q4.3 (D)
- net W_OUT: now also D8.1 (K)
- new net: C18.1, D5.1 (K), IC2.5 (REF1), IC2.6 (REF2), R15.2
- new net U_SW: C9.1, IC1.18 (SHA), IC2.3 (INP), Q1.1 (S), Q2.3 (D), R16.1
- new net V_SW: C10.1, IC1.15 (SHB), IC2.7 (INP), Q3.1 (S), Q4.3 (D), R29.1
Other:
- removed sheet Phase A Current Sense
- removed sheet sheet613E4E23
- note added: "Casting Planeshift"
